File: PCB-Project/PCB-Project.kicad_sch (KiCad schematic)
At the start: 32 parts, among them Q1 AO3401A, SW1 SW_SPDT, U1 STM32F405RGT6, U2 MP2359DJ-LF-Z-MS, Y1 16MHz

Commit message: Schematic updated
Parts:
- added C16: 0u1, symbol Device:C_Small
- added J1: Screw_Terminal_01x02, symbol Connector:Screw_Terminal_01x02
- added J2: SWD, symbol Connector_Generic:Conn_02x05_Odd_Even
- added R10, R11, R8, R9: 22, symbol Device:R_Small
Connections:
- net +12V: now also J1.1 (Pin_1)
- net +3.3V: now also J2.1 (Pin_1)
- net GND: now also C16.2, J1.2 (Pin_2), J2.3 (Pin_3), J2.5 (Pin_5), J2.9 (Pin_9)
- net NRST: now also R11.2
- net SWCLK: now also R9.2
- net SWDIO: now also R8.2
- net SWO: now also R10.2
- new net: J2.4 (Pin_4), R9.1
- new net: J2.6 (Pin_6), R10.1
- new net: C16.1, J2.10 (Pin_10), R11.1
- new net: J2.2 (Pin_2), R8.1
- no-connect marks 39 -> 41
