File: electronics/pcb/design/stm32f405_devboard_v1.0.0.kicad_sch (KiCad schematic)
At the start: 50 parts, among them J1 Screw_Terminal_01x02, J2 SWD, J3 USB_B_Micro, J4 Conn_01x04, J5 Conn_01x04, Q1 AO3401A, SW1 SW_SPDT, U1 STM32F405RGT6, U2 MP2359DJ-LF-Z-MS, U3 USBLC6-2SC6, Y1 16MHz

Commit message: Add schematic to README
Other:
- note added: "Communication Interfaces"
- note added: "Filtering Supply, Clocking & Internal LDO"
- note added: "MICROCONTROLLER"
- note added: "POWER"
- note removed: "Can I use other connector pins for the protocol?"
- note removed: "Connectors and USB"
- note removed: "Power"
- note removed: "Power Entry & Reverse Polarity"
- note removed: "STM32 Microcontroller"
- moved on the sheet: C1, C10, C11, C12, C13, C14, C15, C16, C2, C3, C4, C5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
